File: opensys/openysy.brd (EAGLE design)
At the start: 50 x 55 mm, 11 parts, among them M1 ARDUINO-NANO-3.0, M2 WIRELESS-NRF24L01, X1 USB

Commit message: change board - now v1.0
Parts:
- added LED2: 20mA, led:CHIPLED_1206
- added R1: 200, rcl:R1206
- added R2: 10k, rcl:R1206
- added S1: (no value), Ergaenzung:TASTER-9314_SMD
Connections:
- removed net LED_2: M1.J1.7
- removed net LED_3: M1.J1.8
- new net LED_0: LED2.C, M1.J1.7
- new net N$1: LED2.A, R1.1
- new net N$4: R2.1, S1.2
- new net REG: M1.J1.8, S1.1
- net GND: now also R1.2, R2.2, S1.3
Routing:
- net GND: track 81.6 -> 215.3 mm
- net LED_0: track 0.00 -> 19.1 mm
- net N$4: track 0.00 -> 5.81 mm
- net REG: track 0.00 -> 4.13 mm
- net N$1: track 0.00 -> 3.18 mm
- net CSN: track 50.8 -> 51.5 mm
Changed lines of the file:
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@@
 <layer number="48" name="Document" color="7" fill="1" visible="yes" active="yes"/>
 <layer number="49" name="Reference" color="7" fill="1" visible="yes" active="yes"/>
+<layer number="50" name="dxf" color="7" fill="1" visible="no" active="yes"/>
 <layer number="51" name="tDocu" color="7" fill="1" visible="yes" active="yes"/>
 <layer number="52" name="bDocu" color="7" fill="1" visible="yes" active="yes"/>
@@
 <layer number="97" name="Info" color="7" fill="1" visible="no" active="no"/>
 <layer number="98" name="Guide" color="6" fill="1" visible="no" active="no"/>
+<layer number="100" name="Muster" color="7" fill="1" visible="no" active="no"/>
 <layer number="101" name="Hidden" color="15" fill="1" visible="yes" active="yes"/>
 <layer number="102" name="Changes" color="12" fill="1" visible="yes" active="yes"/>
+<layer number="104" name="S_DOKU" color="7" fill="1" visible="no" active="yes"/>
+<layer number="199" name="Contour" color="7" fill="1" visible="no" active="yes"/>
+<layer number="200" name="200bmp" color="1" fill="10" visible="no" active="no"/>
+<layer number="250" name="Descript" color="3" fill="1" visible="no" active="no"/>
+<layer number="251" name="SMDround" color="12" fill="11" visible="no" active="no"/>
+<layer number="254" name="OrgLBR" color="13" fill="1" visible="no" active="yes"/>
 </layers>
 <board>
@@
 <element name="R4" library="rcl" package="R1206" value="200" x="40.64" y="10.16" rot="MR90"/>
 <element name="LED1" library="led" package="CHIPLED_1206" value="20mA" x="38.1" y="5.08" rot="MR270"/>
+<element name="R1" library="rcl" package="R1206" value="200" x="33.02" y="38.1" smashed="yes" rot="MR90">
+<attribute name="NAME" x="30.48" y="34.29" size="1.27" layer="26" rot="MR90"/>
+</element>
+<element name="LED2" library="led" package="CHIPLED_1206" value="20mA" x="33.02" y="31.75" rot="MR180"/>
+<element name="S1" library="Ergaenzung" package="TASTER-9314_SMD" value="" x="38.1" y="29.21" rot="MR90"/>
+<element name="R2" library="rcl" package="R1206" value="10k" x="35.56" y="38.1" smashed="yes" rot="MR90">
+<attribute name="NAME" x="36.83" y="35.56" size="1.27" layer="26" rot="MR90"/>
+</element>
 </elements>
 <signals>
@@
 <contactref element="R4" pad="2"/>
 <wire x1="40.64" y1="11.582" x2="40.64" y2="13.97" width="0.4064" layer="16"/>
+<contactref element="R1" pad="2"/>
+<wire x1="21.59" y1="44.58" x2="22.73" y2="44.58" width="0.4064" layer="16"/>
+<wire x1="22.73" y1="44.58" x2="26.67" y2="40.64" width="0.4064" layer="16"/>
+<wire x1="26.67" y1="40.64" x2="31.902" y2="40.64" width="0.4064" layer="16"/>
+<wire x1="31.902" y1="40.64" x2="33.02" y2="39.522" width="0.4064" layer="16"/>
+<contactref element="S1" pad="3"/>
+<contactref element="R2" pad="2"/>
+<wire x1="33.02" y1="39.522" x2="35.56" y2="39.522" width="0.4064" layer="16"/>
+<wire x1="35.85" y1="24.21" x2="39.58" y2="27.94" width="0.4064" layer="16"/>
+<wire x1="39.58" y1="27.94" x2="45.72" y2="27.94" width="0.4064" layer="16"/>
+<wire x1="45.72" y1="27.94" x2="48.26" y2="25.4" width="0.4064" layer="16"/>
+<wire x1="48.26" y1="25.4" x2="48.26" y2="5.08" width="0.4064" layer="16"/>
+<wire x1="48.26" y1="5.08" x2="44.45" y2="1.27" width="0.4064" layer="16"/>
+<wire x1="44.45" y1="1.27" x2="17.78" y2="1.27" width="0.4064" layer="16"/>
+<wire x1="17.78" y1="1.27" x2="8.89" y2="10.16" width="0.4064" layer="16"/>
+<wire x1="8.89" y1="10.16" x2="3.81" y2="10.16" width="0.4064" layer="16"/>
+<wire x1="3.81" y1="10.16" x2="2.54" y2="11.43" width="0.4064" layer="16"/>
+<wire x1="2.54" y1="11.43" x2="2.54" y2="31.75" width="0.4064" layer="16"/>
+<wire x1="2.54" y1="31.75" x2="5.08" y2="34.29" width="0.4064" layer="16"/>
+<wire x1="5.08" y1="34.29" x2="8.89" y2="34.29" width="0.4064" layer="16"/>
+<wire x1="8.89" y1="34.29" x2="10.29" y2="32.89" width="0.4064" layer="16"/>
+<wire x1="10.29" y1="32.89" x2="10.29" y2="31.75" width="0.4064" layer="16"/>
 </signal>
 <signal name="CE">
@@
 <contactref element="M2" pad="4"/>
 <contactref element="M1" pad="J1.13"/>
-<wire x1="25.4" y1="38.1" x2="36.83" y2="38.1" width="0.4064" layer="16"/>
-<wire x1="36.83" y1="38.1" x2="41.91" y2="33.02" width="0.4064" layer="16"/>
-<wire x1="41.91" y1="33.02" x2="46.99" y2="33.02" width="0.4064" layer="16"/>
+<wire x1="25.4" y1="38.1" x2="39.37" y2="38.1" width="0.4064" layer="16"/>
 <wire x1="46.99" y1="33.02" x2="48.26" y2="34.29" width="0.4064" layer="16"/>
 <wire x1="48.26" y1="34.29" x2="48.26" y2="35.56" width="0.4064" layer="16"/>
@@
 <wire x1="21.59" y1="39.37" x2="24.13" y2="39.37" width="0.4064" layer="16"/>
 <wire x1="24.13" y1="39.37" x2="25.4" y2="38.1" width="0.4064" layer="16"/>
+<wire x1="39.37" y1="38.1" x2="41.91" y2="35.56" width="0.4064" layer="16"/>
+<wire x1="41.91" y1="35.56" x2="41.91" y2="34.29" width="0.4064" layer="16"/>
+<wire x1="41.91" y1="34.29" x2="43.18" y2="33.02" width="0.4064" layer="16"/>
+<wire x1="43.18" y1="33.02" x2="46.99" y2="33.02" width="0.4064" layer="16"/>
 </signal>
 <signal name="SCK">
@@
 <wire x1="16.51" y1="43.18" x2="20.19" y2="43.18" width="0.4064" layer="16"/>
 <wire x1="20.19" y1="43.18" x2="21.59" y2="41.78" width="0.4064" layer="16"/>
-<wire x1="21.59" y1="41.78" x2="26.8" y2="41.78" width="0.4064" layer="16"/>
-<wire x1="26.8" y1="41.78" x2="29.21" y2="39.37" width="0.4064" layer="16"/>
 <wire x1="16.51" y1="43.18" x2="16.51" y2="38.23" width="0.4064" layer="16"/>
 <wire x1="16.51" y1="38.23" x2="16.64" y2="38.1" width="0.4064" layer="16"/>
+<wire x1="21.59" y1="41.78" x2="22.99" y2="41.78" width="0.4064" layer="16"/>
+<wire x1="22.99" y1="41.78" x2="25.4" y2="39.37" width="0.4064" layer="16"/>
+<wire x1="25.4" y1="39.37" x2="29.21" y2="39.37" width="0.4064" layer="16"/>
 </signal>
 <signal name="1">
@@
 <wire x1="20.32" y1="36.83" x2="22.86" y2="36.83" width="0.4064" layer="16"/>
 </signal>
-<signal name="LED_2">
+<signal name="LED_0">
 <contactref element="M1" pad="J1.7"/>
-</signal>
-<signal name="LED_3">
+<contactref element="LED2" pad="C"/>
+<wire x1="44.45" y1="21.59" x2="34.29" y2="21.59" width="0.4064" layer="16"/>
+<wire x1="34.29" y1="21.59" x2="33.02" y2="22.86" width="0.4064" layer="16"/>
+<wire x1="33.02" y1="22.86" x2="33.02" y2="30" width="0.4064" layer="16"/>
+</signal>
+<signal name="REG">
 <contactref element="M1" pad="J1.8"/>
+<contactref element="S1" pad="1"/>
+<wire x1="40.35" y1="24.21" x2="40.43" y2="24.13" width="0.4064" layer="16"/>
+<wire x1="40.43" y1="24.13" x2="44.45" y2="24.13" width="0.4064" layer="16"/>
 </signal>
 <signal name="LED_4">
@@
 <wire x1="40.64" y1="5.87" x2="40.64" y2="8.738" width="0.4064" layer="16"/>
 </signal>
+<signal name="N$1">
+<contactref element="R1" pad="1"/>
+<contactref element="LED2" pad="A"/>
+<wire x1="33.02" y1="33.5" x2="33.02" y2="36.678" width="0.4064" layer="16"/>
+</signal>
+<signal name="N$4">
+<contactref element="S1" pad="2"/>
+<contactref element="R2" pad="1"/>
+<wire x1="35.56" y1="36.678" x2="37.882" y2="36.678" width="0.4064" layer="16"/>
+<wire x1="37.882" y1="36.678" x2="40.35" y2="34.21" width="0.4064" layer="16"/>
+</signal>
 </signals>

Commit message: smart home platine now v3
lets try it now
Parts:
- removed R3, R5: 0, rcl:R1206
- removed X1: USB, con-berg:PN87520
- added JP2: VCC, pinhead:1X02
- added LED3, LED4, LED5: 20mA, led:CHIPLED_1206
- added R6, R7, R8: 200, rcl:R1206
- added X2: USBPTH, usb:USB-B-PTH
- S1: value (none) -> S1
- moved R1 31.0 mm to (32.1, 7.14)
- moved LED2 24.5 mm to (32.4, 7.26), flipped to the top, turned to 0 degrees
- moved S1 22.5 mm to (26.0, 10.2), flipped to the top
- moved R2 18.2 mm to (43.0, 21.5), turned to 180 degrees
- moved C1 12.8 mm to (10.2, 37.3)
- moved JP1 8.03 mm to (25.4, 33.0)
- moved M1 8.03 mm to (39.4, 31.8)
- moved R4 5.71 mm to (35.8, 7.09)
- moved LED1 2.99 mm to (36.1, 7.26), flipped to the top, turned to 0 degrees
- moved C2 1.39 mm to (10.2, 32.1), turned to 270 degrees
- moved C3 0.62 mm to (15.2, 38.7)
Connections:
- net LED_0 renamed LED_TX
- removed net CE-TMP: M2.3, R3.2
- removed net LED_4: M1.J1.9
- removed net LED_5: M1.J1.10
- removed net LED_6: M1.J1.11
- removed net N$3: JP1.1, R5.1
- new net LED_1: LED3.C, M1.J1.9
- new net LED_2: LED4.C, M1.J1.10
- new net LED_3: LED5.C, M1.J1.11
- new net N$5: LED3.A, R6.1
- new net N$6: LED4.A, R7.1
- new net N$7: LED5.A, R8.1
- net CE: now also M2.3; no longer R3.1
- net GND: now also JP2.2, R6.2, R7.2, R8.2, X2.GND; no longer S1.3, X1.4
- net VCC: now also JP1.1, JP2.1, S1.3, X2.VBUS; no longer R5.2, X1.1
Routing:
- net GND: track 215.3 -> 137.4 mm
- net REG: track 4.13 -> 45.2 mm
- net LED_2: track 0.00 -> 36.6 mm, vias 0 -> 1
- net LED_1: track 0.00 -> 36.3 mm, vias 0 -> 2
- net LED_3: track 0.00 -> 31.8 mm
- net MOSI: track 67.2 -> 38.2 mm
- net CE: track 22.9 -> 49.5 mm, vias 0 -> 1
- net N$4: track 5.81 -> 22.1 mm, vias 0 -> 1
- net N$3: track 15.3 -> 0.00 mm
- net CSN: track 51.5 -> 36.5 mm, vias 0 -> 1
- net LED_TX: track 19.1 -> 33.6 mm
- net CE-TMP: track 12.3 -> 0.00 mm
- net +3V3: track 19.4 -> 28.9 mm
- net VCC: track 91.1 -> 99.5 mm, vias 0 -> 5
- net N$5: track 0.00 -> 4.88 mm, vias 0 -> 1
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