File: opensys/openysy.sch (EAGLE design)
At the start: 11 parts, among them M1 ARDUINO-NANO-3.0, M2 WIRELESS-NRF24L01, X1 USB

Commit message: change board - now v1.0
Parts:
- added LED2: 20mA, led:LEDCHIPLED_1206
- added R1: 200, rcl:R-EU_R1206
- added R2: 10k, rcl:R-EU_R1206
- added S1: (no value), Ergaenzung:TASTER-9314_SMD
Connections:
- removed net LED_2: M1.D4
- removed net LED_3: M1.D5
- new net LED_0: LED2.C, M1.D4
- new net N$1: LED2.A, R1.1
- new net N$4: R2.1, S1.2
- new net REG: M1.D5, S1.1
- net GND: now also R1.2, R2.2, S1.3
Other:
- moved on the sheet: JP1, R5
Changed lines of the file:
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@@
 <layer number="48" name="Document" color="7" fill="1" visible="no" active="no"/>
 <layer number="49" name="Reference" color="7" fill="1" visible="no" active="no"/>
+<layer number="50" name="dxf" color="7" fill="1" visible="no" active="no"/>
 <layer number="51" name="tDocu" color="7" fill="1" visible="no" active="no"/>
 <layer number="52" name="bDocu" color="7" fill="1" visible="no" active="no"/>
@@
 <layer number="97" name="Info" color="7" fill="1" visible="yes" active="yes"/>
 <layer number="98" name="Guide" color="6" fill="1" visible="yes" active="yes"/>
+<layer number="100" name="Muster" color="7" fill="1" visible="no" active="no"/>
 <layer number="101" name="Hidden" color="15" fill="1" visible="yes" active="yes"/>
 <layer number="102" name="Changes" color="12" fill="1" visible="yes" active="yes"/>
+<layer number="104" name="S_DOKU" color="7" fill="1" visible="no" active="yes"/>
+<layer number="199" name="Contour" color="7" fill="1" visible="no" active="yes"/>
+<layer number="200" name="200bmp" color="1" fill="10" visible="no" active="no"/>
+<layer number="250" name="Descript" color="3" fill="1" visible="no" active="no"/>
+<layer number="251" name="SMDround" color="12" fill="11" visible="no" active="no"/>
+<layer number="254" name="OrgLBR" color="13" fill="1" visible="no" active="yes"/>
 </layers>
 <schematic xreflabel="%F%N/%S.%C%R" xrefpart="/%S.%C%R">
@@
 <part name="GND6" library="supply1" deviceset="GND" device=""/>
 <part name="LED1" library="led" deviceset="LED" device="CHIPLED_1206" value="20mA"/>
+<part name="R1" library="rcl" deviceset="R-EU_" device="R1206" value="200"/>
+<part name="GND7" library="supply1" deviceset="GND" device=""/>
+<part name="LED2" library="led" deviceset="LED" device="CHIPLED_1206" value="20mA"/>
+<part name="S1" library="Ergaenzung" deviceset="TASTER-9314_SMD" device=""/>
+<part name="GND8" library="supply1" deviceset="GND" device=""/>
+<part name="R2" library="rcl" deviceset="R-EU_" device="R1206" value="10k"/>
+<part name="GND9" library="supply1" deviceset="GND" device=""/>
 </parts>
 <sheets>
@@
 <instance part="+3V2" gate="G$1" x="132.08" y="76.2" rot="R270"/>
 <instance part="C3" gate="G$1" x="127" y="71.12"/>
-<instance part="JP1" gate="A" x="132.08" y="15.24"/>
-<instance part="GND5" gate="1" x="121.92" y="-2.54"/>
-<instance part="P+3" gate="VCC" x="101.6" y="25.4" rot="R90"/>
+<instance part="JP1" gate="A" x="139.7" y="22.86"/>
+<instance part="GND5" gate="1" x="129.54" y="5.08"/>
+<instance part="P+3" gate="VCC" x="109.22" y="33.02" rot="R90"/>
 <instance part="R3" gate="G$1" x="132.08" y="83.82" rot="R180"/>
-<instance part="R5" gate="G$1" x="111.76" y="25.4" rot="R180"/>
+<instance part="R5" gate="G$1" x="119.38" y="33.02" rot="R180"/>
 <instance part="R4" gate="G$1" x="154.94" y="63.5" rot="R270"/>
 <instance part="GND6" gate="1" x="154.94" y="53.34"/>
 <instance part="LED1" gate="G$1" x="154.94" y="73.66" rot="R180"/>
+<instance part="R1" gate="G$1" x="167.64" y="63.5" rot="R270"/>
+<instance part="GND7" gate="1" x="167.64" y="53.34"/>
+<instance part="LED2" gate="G$1" x="167.64" y="73.66" rot="R180"/>
+<instance part="S1" gate="G$1" x="154.94" y="33.02"/>
+<instance part="GND8" gate="1" x="149.86" y="20.32"/>
+<instance part="R2" gate="G$1" x="167.64" y="33.02" rot="R270"/>
+<instance part="GND9" gate="1" x="167.64" y="20.32"/>
 </instances>
 <busses>
@@
 <pinref part="R5" gate="G$1" pin="2"/>
 <pinref part="P+3" gate="VCC" pin="VCC"/>
-<wire x1="104.14" y1="25.4" x2="106.68" y2="25.4" width="0.1524" layer="91"/>
+<wire x1="111.76" y1="33.02" x2="114.3" y2="33.02" width="0.1524" layer="91"/>
 </segment>
 <segment>
@@
 <pinref part="GND5" gate="1" pin="GND"/>
 <pinref part="JP1" gate="A" pin="10"/>
-<wire x1="121.92" y1="0" x2="121.92" y2="2.54" width="0.1524" layer="91"/>
-<wire x1="121.92" y1="2.54" x2="129.54" y2="2.54" width="0.1524" layer="91"/>
+<wire x1="129.54" y1="7.62" x2="129.54" y2="10.16" width="0.1524" layer="91"/>
+<wire x1="129.54" y1="10.16" x2="137.16" y2="10.16" width="0.1524" layer="91"/>
 </segment>
 <segment>
@@
 <pinref part="GND6" gate="1" pin="GND"/>
 <wire x1="154.94" y1="58.42" x2="154.94" y2="55.88" width="0.1524" layer="91"/>
+</segment>
+<segment>
+<pinref part="R1" gate="G$1" pin="2"/>
+<pinref part="GND7" gate="1" pin="GND"/>
+<wire x1="167.64" y1="58.42" x2="167.64" y2="55.88" width="0.1524" layer="91"/>
+</segment>
+<segment>
+<pinref part="GND8" gate="1" pin="GND"/>
+<pinref part="S1" gate="G$1" pin="3"/>
+<wire x1="149.86" y1="22.86" x2="149.86" y2="27.94" width="0.1524" layer="91"/>
+</segment>
+<segment>
+<pinref part="GND9" gate="1" pin="GND"/>
+<pinref part="R2" gate="G$1" pin="2"/>
+<wire x1="167.64" y1="22.86" x2="167.64" y2="27.94" width="0.1524" layer="91"/>
 </segment>
 </net>
@@
 <segment>
 <pinref part="JP1" gate="A" pin="2"/>
-<wire x1="129.54" y1="22.86" x2="116.84" y2="22.86" width="0.1524" layer="91"/>
-<label x="116.84" y="22.86" size="1.778" layer="95"/>
+<wire x1="137.16" y1="30.48" x2="124.46" y2="30.48" width="0.1524" layer="91"/>
+<label x="124.46" y="30.48" size="1.778" layer="95"/>
 </segment>
 <segment>
@@
 <segment>
 <pinref part="JP1" gate="A" pin="3"/>
-<wire x1="129.54" y1="20.32" x2="116.84" y2="20.32" width="0.1524" layer="91"/>
-<label x="116.84" y="20.32" size="1.778" layer="95"/>
+<wire x1="137.16" y1="27.94" x2="124.46" y2="27.94" width="0.1524" layer="91"/>
+<label x="124.46" y="27.94" size="1.778" layer="95"/>
 </segment>
 <segment>
@@
 <segment>
 <pinref part="JP1" gate="A" pin="4"/>
-<wire x1="129.54" y1="17.78" x2="116.84" y2="17.78" width="0.1524" layer="91"/>
-<label x="116.84" y="17.78" size="1.778" layer="95"/>
+<wire x1="137.16" y1="25.4" x2="124.46" y2="25.4" width="0.1524" layer="91"/>
+<label x="124.46" y="25.4" size="1.778" layer="95"/>
 </segment>
 <segment>
@@
 <segment>
 <pinref part="JP1" gate="A" pin="5"/>
-<wire x1="129.54" y1="15.24" x2="116.84" y2="15.24" width="0.1524" layer="91"/>
-<label x="116.84" y="15.24" size="1.778" layer="95"/>
+<wire x1="137.16" y1="22.86" x2="124.46" y2="22.86" width="0.1524" layer="91"/>
+<label x="124.46" y="22.86" size="1.778" layer="95"/>
 </segment>
 <segment>
@@
 <segment>
 <pinref part="JP1" gate="A" pin="6"/>
-<wire x1="129.54" y1="12.7" x2="116.84" y2="12.7" width="0.1524" layer="91"/>
-<label x="116.84" y="12.7" size="1.778" layer="95"/>
+<wire x1="137.16" y1="20.32" x2="124.46" y2="20.32" width="0.1524" layer="91"/>
+<label x="124.46" y="20.32" size="1.778" layer="95"/>
 </segment>
 <segment>
@@
 <segment>
 <pinref part="JP1" gate="A" pin="7"/>
-<wire x1="129.54" y1="10.16" x2="116.84" y2="10.16" width="0.1524" layer="91"/>
-<label x="116.84" y="10.16" size="1.778" layer="95"/>
+<wire x1="137.16" y1="17.78" x2="124.46" y2="17.78" width="0.1524" layer="91"/>
+<label x="124.46" y="17.78" size="1.778" layer="95"/>
 </segment>
 <segment>
@@
 <segment>
 <pinref part="JP1" gate="A" pin="8"/>
-<wire x1="129.54" y1="7.62" x2="116.84" y2="7.62" width="0.1524" layer="91"/>
-<label x="116.84" y="7.62" size="1.778" layer="95"/>
+<wire x1="137.16" y1="15.24" x2="124.46" y2="15.24" width="0.1524" layer="91"/>
+<label x="124.46" y="15.24" size="1.778" layer="95"/>
 </segment>
 <segment>
@@
 <segment>
 <pinref part="JP1" gate="A" pin="9"/>
-<wire x1="129.54" y1="5.08" x2="116.84" y2="5.08" width="0.1524" layer="91"/>
-<label x="116.84" y="5.08" size="1.778" layer="95"/>
+<wire x1="137.16" y1="12.7" x2="124.46" y2="12.7" width="0.1524" layer="91"/>
+<label x="124.46" y="12.7" size="1.778" layer="95"/>
 </segment>
 <segment>
@@
 <segment>
 <pinref part="JP1" gate="A" pin="1"/>
-<wire x1="116.84" y1="25.4" x2="129.54" y2="25.4" width="0.1524" layer="91"/>
+<wire x1="124.46" y1="33.02" x2="137.16" y2="33.02" width="0.1524" layer="91"/>
 <pinref part="R5" gate="G$1" pin="1"/>
 </segment>
 </net>
-<net name="LED_2" class="0">
+<net name="LED_0" class="0">
 <segment>
 <pinref part="M1" gate="G$1" pin="D4"/>
@@
 <label x="17.78" y="35.56" size="1.778" layer="95"/>
 </segment>
-</net>
-<net name="LED_3" class="0">
+<segment>
+<pinref part="LED2" gate="G$1" pin="C"/>
+<wire x1="167.64" y1="78.74" x2="167.64" y2="81.28" width="0.1524" layer="91"/>
+<label x="167.64" y="81.28" size="1.778" layer="95"/>
+</segment>
+</net>
+<net name="REG" class="0">
 <segment>
 <pinref part="M1" gate="G$1" pin="D5"/>
@@
 <label x="17.78" y="33.02" size="1.778" layer="95"/>
 </segment>
+<segment>
+<pinref part="S1" gate="G$1" pin="1"/>
+<wire x1="149.86" y1="38.1" x2="147.32" y2="38.1" width="0.1524" layer="91"/>
+<label x="144.78" y="38.1" size="1.778" layer="95"/>
+</segment>
 </net>
 <net name="LED_4" class="0">
@@
 </segment>
 </net>
+<net name="N$1" class="0">
+<segment>
+<pinref part="R1" gate="G$1" pin="1"/>
+<pinref part="LED2" gate="G$1" pin="A"/>
+<wire x1="167.64" y1="71.12" x2="167.64" y2="68.58" width="0.1524" layer="91"/>
+</segment>
+</net>
+<net name="N$4" class="0">
+<segment>
+<pinref part="S1" gate="G$1" pin="2"/>
+<pinref part="R2" gate="G$1" pin="1"/>
+<wire x1="160.02" y1="38.1" x2="167.64" y2="38.1" width="0.1524" layer="91"/>
+</segment>
+</net>

Commit message: smart home platine now v3
lets try it now
Parts:
- removed R3, R5: 0, rcl:R-EU_R1206
- removed X1: USB, con-berg:PN87520
- added JP2: VCC, pinhead:PINHD-1X2
- added LED3, LED4, LED5: 20mA, led:LEDCHIPLED_1206
- added R6, R7, R8: 200, rcl:R-EU_R1206
- added X2: USBPTH, usb:USBPTH
- S1: value (none) -> S1
Connections:
- net LED_0 renamed LED_TX
- removed net CE-TMP: M2.CE, R3.2
- removed net LED_4: M1.D6
- removed net LED_5: M1.D7
- removed net LED_6: M1.D8
- removed net N$3: JP1.1, R5.1
- new net LED_1: LED3.C, M1.D6
- new net LED_2: LED4.C, M1.D7
- new net LED_3: LED5.C, M1.D8
- new net N$5: LED3.A, R6.1
- new net N$6: LED4.A, R7.1
- new net N$7: LED5.A, R8.1
- net CE: now also M2.CE; no longer R3.1
- net GND: now also JP2.2, R6.2, R7.2, R8.2, X2.GND; no longer S1.3, X1.4
- net VCC: now also JP1.1, JP2.1, S1.3, X2.VBUS; no longer R5.2, X1.1
Other:
- moved on the sheet: C2
